File: PCB/Eros/Eros.kicad_sch (KiCad schematic)
At the start: 99 parts, among them J1 USB_C_PowerOnly_6P, J2 UART, J3 Li-ion, J4 Conn_01x08_Socket, J6 Micro_SD_Card, Q1 BC817, SW1 SW_Push, SW2 SW_Push, SW3 SW_Push, SW4 SW_Push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

Commit message: Poprawinie footprintów oraz naprawienie błędów ERC
Parts:
- removed R32, R33: 4.7k, Resistor_SMD:R_0402_1005Metric_Pad0.72x0.64mm_HandSolder, symbol Device:R
- removed SW1, SW2: SW_Push, Button_Switch_SMD:SW_Push_1P1T_NO_CK_KMR2, symbol Switch:SW_Push
- removed U2: LIS3DH, Package_LGA:LGA-16_3x3mm_P0.5mm_LayoutBorder3x5y, symbol Sensor_Motion:LIS3DH
- added SW1, SW2: SW_Push, Button_Switch_SMD:SW_Push_1P1T-SH_NO_CK_KMR2xxG, symbol Moje_symbole:SW_Push
- added U2: LIS3DH, Package_LGA:LGA-16_3x3mm_P0.5mm_LayoutBorder3x5y, symbol Moje_symbole:LIS3DH
- C24, C25: value 0.1u -> 100n
- R26: footprint Resistor_SMD:R_0402_1005Metric_Pad0.72x0.64mm_HandSolder -> Resistor_SMD:R_0805_2012Metric_Pad1.20x1.40mm_HandSolder
Connections:
- net +3.3V: now also U2.1 (VDD_IO), U2.14 (VDD), U2.8 (CS)
- net BOOT: now also SW1.1
- net GND: now also SW1.2, SW1.SH, SW2.2, SW2.SH, U2.10 (GND), U2.12 (GND), U2.5 (GND), U2.7 (SDO); no longer SW3.1, SW4.1, SW5.1
- net RESET: now also SW2.1
- net RTC_GPIO: now also U2.11 (INT1)
- net SCL1: now also U2.4 (SPC)
- net SDA1: now also U2.6 (SDI)
- net SDN: now also U1.8 (IO32)
- net SCL2: no longer names the net of U1.28 (IO17)
- net SDA2: no longer names the net of U1.27 (IO16)
- no-connect marks 11 -> 12
Other:
- note added: "Jula dodaj power supply supervisor i poczytaj o bms (baterry management systems)!!! ZROBIŁAM"
- note removed: "Filtr górno przepustowy to kondensatory C22 i C23. Odcinają one 0.5Hz. Człowiek jak się porusza ma około 1.5-2Hz a jak śpi to około 0.7Hz. Można zmienić te kondensatory tak aby odcinały 1Hz lub więcej. Ale jest to kompromis. Usuniemy szumy przy ruchu, ale w spoczynku nie będzie tak szczegółowego wykresu z detalami (ale bicie serca będzie dalej dobrze odczytywalne). Kompromisem jest np. 0.7Hz i pr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"
- note removed: "Jula dodaj power supply supervisor i poczytaj o bms (baterry management systems)!!! TEGO JESZCZE NIE ZROBIŁAM"
- note removed: "Kurde jednak myślę że można zostawić te 0.5Hz i programowo akurat to wyłapywać."
