File: PCB/Eros/Eros.kicad_sch (KiCad schematic)
At the start: 107 parts, among them J1 USB_C_PowerOnly_6P, J2 UART, J3 Li-ion, J4 Conn_01x08_Socket, J5 Conn_01x03_Socket, J6 Micro_SD_Card, J7 AudioJack3, Q1 BC817, SW1 SW_Push, SW2 SW_Push, SW3 SW_Push, SW4 SW_Push, SW5 SW_Push, SW6 SW_SPDT, U1 ESP32-WROOM-32E, U2 LIS3DH, U3 MCP73831-2-OT, U4 AP2112K-3.3, U5 ADS1115IDGS, U6 MCP100-315D, U7 AD8232, U8 OPA333xxD

Commit message: Poprawa schematu oraz ulozenie komponentow
Parts:
- removed C4: 100n, Capacitor_SMD:C_0402_1005Metric_Pad0.74x0.62mm_HandSolder, symbol Device:C
- removed J5: Conn_01x03_Socket, Connector_PinHeader_1.27mm:PinHeader_1x03_P1.27mm_Vertical, symbol Connector:Conn_01x03_Socket
- removed J7: AudioJack3, Connector_Audio:Jack_3.5mm_Lumberg_1503_03_Horizontal, symbol Connector_Audio:AudioJack3
- removed JP3, JP4: SolderJumper_2_Open, Jumper:SolderJumper-2_P1.3mm_Open_Pad1.0x1.5mm, symbol Jumper:SolderJumper_2_Open
- removed R29, R30: R, Resistor_SMD:R_0402_1005Metric_Pad0.72x0.64mm_HandSolder, symbol Device:R
- removed R32, R4: 10k, Resistor_SMD:R_0402_1005Metric_Pad0.72x0.64mm_HandSolder, symbol Device:R
- removed R34: 10k, Resistor_SMD:R_01005_0402Metric_Pad0.57x0.30mm_HandSolder, symbol Device:R
- removed SW3: SW_Push, Button_Switch_THT:SW_Tactile_SPST_Angled_PTS645Vx39-2LFS, symbol Switch:SW_Push
- removed TP6: TestPoint, TestPoint:TestPoint_Pad_D1.5mm, symbol Connector:TestPoint
- removed U5: ADS1115IDGS, Package_SO:TSSOP-10_3x3mm_P0.5mm, symbol Analog_ADC:ADS1115IDGS
- removed U7: AD8232, AD8232:QFN-20_EP_4x4_Pitch0.5mm, symbol AD8232:AD8232ACPZ
- removed U8: OPA333xxD, Package_SO:SOIC-8_3.9x4.9mm_P1.27mm, symbol Amplifier_Operational:OPA333xxD
- added C31, C35, C39, C41: 100n, Capacitor_SMD:C_0402_1005Metric_Pad0.74x0.62mm_HandSolder, symbol Device:C
- added C32, C33: 1n, Capacitor_SMD:C_0402_1005Metric_Pad0.74x0.62mm_HandSolder, symbol Device:C
- added C34: 1.5n, Capacitor_SMD:C_0402_1005Metric_Pad0.74x0.62mm_HandSolder, symbol Device:C
- added C36: 10u, Capacitor_SMD:C_0603_1608Metric_Pad1.08x0.95mm_HandSolder, symbol Device:C
- added C37, C38: 47p, Capacitor_SMD:C_0402_1005Metric_Pad0.74x0.62mm_HandSolder, symbol Device:C
- added C40, C42: 1u, Capacitor_SMD:C_0402_1005Metric_Pad0.74x0.62mm_HandSolder, symbol Device:C
- added D1, D4, D5, D6: BAV99, Package_TO_SOT_SMD:SOT-23, symbol Diode:BAV99
- added FB2: FerriteBead(600om), Inductor_SMD:L_0402_1005Metric_Pad0.77x0.64mm_HandSolder, symbol Device:FerriteBead
- added IC1: ADS1292RIPBS, ADS1292:QFP50P700X700X120-32N, symbol ADS1292RIPBS:ADS1292RIPBS
- added J5: AudioJack3, Connector_Audio:Jack_3.5mm_Lumberg_1503_03_Horizontal, symbol Connector_Audio:AudioJack3
- added J7: Conn_01x03_Socket, Connector_PinHeader_2.54mm:PinHeader_1x03_P2.54mm_Vertical, symbol Connector:Conn_01x03_Socket
- added R33: 10k, Resistor_SMD:R_0402_1005Metric_Pad0.72x0.64mm_HandSolder, symbol Device:R
- C19: value 1n -> 47n
- C20: value 10n -> 47n
- C21: value 1.5n -> 2.2u
- C22: value 0.33u -> 2.2u
- C23: value 0.33u -> 22u
- C26, C27: value C -> 2.2n; now fitted
- C29, C30: value 100n -> 2.2n
- FB1: value FerriteBead -> FerriteBead(120om)
- J3: footprint BHC-18650-1P COMF:BatteryHolder_MPD_BH-18650-PC -> Connector_JST:JST_PH_B2B-PH-K_1x02_P2.00mm_Vertical
- R15: value 180k -> 10k
- R16: value 180k -> 10M
- R18: value 10M -> 40.2k
- R19: value 360k -> 51k
- R20: value 100k -> 40.2k
- R21: value 1M -> 51k
- R22, R23: value 1M -> 10M
- R24: value 10M -> 1M
- R25, R27: value 10M -> 100k
- R26: value 1.4M -> 0R; footprint Resistor_SMD:R_0805_2012Metric_Pad1.20x1.40mm_HandSolder -> Resistor_SMD:R_0402_1005Metric_Pad0.72x0.64mm_HandSolder
- R28: value 10M -> 10k
- R31: footprint Resistor_SMD:R_01005_0402Metric_Pad0.57x0.30mm_HandSolder -> Resistor_SMD:R_0402_1005Metric_Pad0.72x0.64mm_HandSolder
- U1: footprint RF_Module:ESP32-WROOM-32D -> RF_Module:ESP32-WROOM-32E
Connections:
- net ADC1 is gone; now on net ADC: C18.1, R13.1, R14.1
- net BUTTON_3 is gone; now on net BUZZER: U1.12 (IO27)
- net SDN is gone; now on net VSPI_CS: U1.8 (IO32)
- net +3.3V: now also R15.1, C41.2, C42.2, FB2.2, IC1.14 (CLKSEL), IC1.23 (DVDD), R33.2; no longer C24.2, C29.1, R17.2, R18.1, R27.2
- net BUTTON_1: now also U1.7 (IO35); no longer U1.10 (IO25)
- net BUTTON_2: now also U1.5 (SENSOR_VN); no longer U1.11 (IO26)
- net BUZZER: no longer U1.7 (IO35)
- net GND: now also C21.2, C22.2, C23.2, C24.2, R17.1, R22.1, R28.1, C32.2, C33.2, C35.2, C36.2, C37.1, C38.2, C39.2, C40.2, C41.1, C42.1, D1.1 (K), D4.1 (K), D5.1 (K), D6.1 (K), IC1.10 (VREFN), IC1.13 (AVSS), IC1.24 (DGND); no longer C24.1, C25.1, C27.1, C29.2, C30.2, R28.2
- net HSPI_CS: now also R15.2, IC1.18 (~{CS}); no longer J4.5 (Pin_5)
- net HSPI_MOSI: now also IC1.19 (DIN); no longer J4.3 (Pin_3)
- net LA: now also C25.1, R19.2, C38.1, J5.R, J7.2 (Pin_2); no longer R15.1, R17.1
- net RA: now also R21.2, C31.1, C37.2, J5.S, J7.1 (Pin_1); no longer R16.1, R18.2
- net RL: now also R25.2, J5.T, J7.3 (Pin_3); no longer R19.1
- net VSPI_CS: now also R33.1; no longer R31.2, U1.29 (IO5)
- net VSPI_MOSI: now also J4.3 (Pin_3)
- net VSPI_SCK: now also J4.4 (Pin_4)
- net at C19.2: now also IC1.1 (PGA1N); no longer R19.2
- net IN1N: now reaches C30.1
- net IN1N: now also R22.2, R23.2, D1.3 (K), IC1.3 (IN1N)
- net RLDINV: now reaches R24.1
- net RLDINV: now also R25.1, R26.1, R27.2, C34.2, IC1.28 (RLDINV); no longer C22.2
- net RLDOUT: now reaches R24.2, R26.2
- net RLDOUT: now also C34.1, IC1.30 (RLDOUT); no longer R25.1
- net VCAP2: now reaches C22.1
- net VCAP2: now also IC1.27 (VCAP2)
- net IN1P: now reaches R16.2
- net IN1P: now also C27.1, R17.2, D5.3 (K), IC1.4 (IN1P)
- net at C19.1: now also IC1.2 (PGA1P)
- net ADC: now reaches U1.4 (SENSOR_VP)
- net HSPI_CLK renamed HSPI_MISO
- net HSPI_MISO: now also IC1.21 (DOUT); no longer J4.4 (Pin_4)
- net IAOUT renamed AVDD
- net AVDD: now also R16.1, C39.1, C40.1, D1.2 (A), D4.2 (A), D5.2 (A), D6.2 (A), FB2.1, IC1.12 (AVDD); no longer R25.2
- net LOD+ renamed HSPI_SCK
- net HSPI_SCK: now also R28.2, IC1.20 (SCLK)
- net LOD- renamed DRDY
- net DRDY: now also IC1.22 (~{DRDY})
- net OPAMP+: no longer names the net of C20.1
- net OPAMP+: now also IC1.8 (PGA2P); no longer R22.2
- net OPAMP-: no longer names the net of R20.1
- net OPAMP-: now also C29.2, C33.1; no longer R21.1
- removed net OUTPUT: C21.2, R21.2
- net REFIN: no longer names the net of C25.2, C27.2
- net REFIN: now also C26.1; no longer R27.1, R28.1
- removed net REFOUT: C20.2, C23.2, C26.2, R20.2
- removed net SW: C23.1, C26.1, R26.1
- new net: C29.1, C30.2, C31.2
- new net: C20.2, IC1.7 (PGA2N)
- new net: C26.2, C32.1, R18.1
- new net DISP_CS: J4.5 (Pin_5), R31.2, U1.29 (IO5)
- new net IN2N: D4.3 (K), IC1.5 (IN2N), R21.1
- new net IN2P: D6.3 (K), IC1.6 (IN2P), R19.1
- new net IN3N: IC1.32 (RESP_MODN/IN3N), R20.2
- new net IN3P: IC1.31 (RESP_MODP/IN3P), R18.2
- new net PWDN: IC1.15 (~{PWDN}/~{RESET}), U1.11 (IO26)
- new net RLDIN: IC1.29 (RLDIN/RLDREF), R27.1
- new net START: IC1.16 (START), U1.10 (IO25)
- new net VCAP1: C21.1, IC1.11 (VCAP1)
- new net VREFP: C23.1, C24.1, C35.1, C36.1, IC1.9 (VREFP)
- no-connect marks 6 -> 8
Other:
- note added: "ADS1292"
- note added: "AFE FILTRING CAPS"
- note added: "ELECTRODES RA & LA"
- note added: "ESD PROTECTION DIODES"
- note added: "MOUNTING HOLES"
- note added: "PORTS FOR ELECTRODES"
- note added: "RLD ELECTRODE"
- note added: "VREF SECTION"
- note removed: "ADC MODULE"
- note removed: "ECG MODULE"
- moved on the sheet: C1, C10, C11, C2, C28, C9, H5, H6, H7, H8, J2, J4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
