File: PCB/Rythmio.kicad_pcb (KiCad board)
At the start: 4 copper layers, 65 x 71 mm, 117 parts, among them IC1 ADS1292RIPBS, J1 USB_C_PowerOnly_6P, J2 UART, J3 Li-ion, J4 Conn_01x08_Socket, J5 AudioJack3, J6 Micro_SD_Card, J7 Conn_01x03_Socket, Q1 BC817, SW1 SW_Push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

Commit message: Rename PCB/ to Rythmio
Parts:
- moved G*** 6.72 mm to (186.5, 54.0)
- moved G*** 2.38 mm to (168.0, 54.0)
Other:
- board text added: "Rythmio"
- board text removed: "EROS"
